Commit message: imported files from v1

File: description/robot.urdf.xacro (robot description, xacro)
@@ -1,35 +1,18 @@
 <?xml version="1.0"?>
 <robot xmlns:xacro="http://www.ros.org/wiki/xacro" name="robot">
-  <link name="base_link"/>
-  <link name="left_wheel_link"/>
-  <link name="right_wheel_link"/>
-  <joint name="left_wheel_joint" type="continuous">
-    <parent link="base_link"/>
-    <child link="left_wheel_link"/>
-    <origin xyz="0 0.15 0" rpy="0 0 0"/>
-    <axis xyz="0 1 0"/>
-  </joint>
-  <joint name="right_wheel_joint" type="continuous">
-    <parent link="base_link"/>
-    <child link="right_wheel_link"/>
-    <origin xyz="0 -0.15 0" rpy="0 0 0"/>
-    <axis xyz="0 1 0"/>
-  </joint>
-  <ros2_control name="ArduinoController" type="system">
-    <hardware>
-      <plugin>halfonso_arduino/SerialArduino</plugin>
-      <param name="port">/dev/ttyUSB0</param>
-      <param name="baud_rate">115200</param>
-    </hardware>
-    <joint name="left_wheel_joint">
-      <command_interface name="velocity"/>
-      <state_interface name="position"/>
-      <state_interface name="velocity"/>
-    </joint>
-    <joint name="right_wheel_joint">
-      <command_interface name="velocity"/>
-      <state_interface name="position"/>
-      <state_interface name="velocity"/>
-    </joint>
-  </ros2_control>
+    <xacro:arg name="use_ros2_control" default="true" />
+    <xacro:arg name="use_ros2_control_gz_sim" default="false" />
+    <!-- Robot_frames -->
+    <xacro:include filename="robot_core.xacro" />
+    <!-- Controls -->
+    <xacro:if value="$(arg use_ros2_control)">
+        <xacro:include filename="ros2_control.xacro" />
+    </xacro:if>
+    <xacro:unless value="$(arg use_ros2_control)">
+        <xacro:include filename="gz_diff_drive_control.xacro" />
+    </xacro:unless>
+    <!-- Sensors -->
+    <xacro:include filename="lidar.xacro" />
+    <!-- <xacro:include filename = "camera.xacro" /> -->
+    <!-- <xacro:include filename = "depth_camera.xacro" /> -->
 </robot>
