Commit message: changes to robot visualization

File: description/robot_core.xacro (robot description, xacro)
@@ -65,5 +65,5 @@
             </geometry> -->
             <geometry>
-                <mesh filename="file://$(find halfonso_v2)/meshes/base_footprint.stl" />
+                <mesh filename="package://halfonso_v2/meshes/base_footprint.stl" />
             </geometry>
             <!-- <material name="orange"/> -->
@@ -82,5 +82,5 @@
             <origin xyz="0 0 0" rpy="0 0 0" />
             <geometry>
-                <mesh filename="file://$(find halfonso_v2)/meshes/base_footprint.stl" />
+                <mesh filename="package://halfonso_v2/meshes/base_footprint.stl" />
             </geometry>
         </collision>
@@ -118,5 +118,5 @@
             </geometry> -->
             <geometry>
-                <mesh filename="file://$(find halfonso_v2)/meshes/base_link.stl" />
+                <mesh filename="package://halfonso_v2/meshes/base_link.stl" />
             </geometry>
             <!-- <material name="orange"/> -->
@@ -136,5 +136,5 @@
             <origin xyz="0 0 0" rpy="0 0 0" />
             <geometry>
-                <mesh filename="file://$(find halfonso_v2)/meshes/base_link.stl" />
+                <mesh filename="package://halfonso_v2/meshes/base_link.stl" />
             </geometry>
         </collision>
@@ -174,5 +174,5 @@
             <geometry>
                 <!-- <cylinder radius="${wheel_radius}" length="${wheel_thickness}"/> -->
-                <mesh filename="file://$(find halfonso_v2)/meshes/left_wheel.stl" />
+                <mesh filename="package://halfonso_v2/meshes/left_wheel.stl" />
             </geometry>
             <!-- <material name="blue"/> -->
@@ -185,5 +185,5 @@
             <geometry>
                 <!-- <sphere radius="${wheel_radius}"/> -->
-                <mesh filename="file://$(find halfonso_v2)/meshes/left_wheel.stl" />
+                <mesh filename="package://halfonso_v2/meshes/left_wheel.stl" />
             </geometry>
         </collision>
@@ -221,5 +221,5 @@
             <origin xyz="0 0 0" rpy="0 0 0" />
             <geometry>
-                <mesh filename="file://$(find halfonso_v2)/meshes/right_wheel.stl" />
+                <mesh filename="package://halfonso_v2/meshes/right_wheel.stl" />
             </geometry>
             <!-- <material name="blue"/> -->
@@ -231,5 +231,5 @@
             <origin xyz="0 0 0" rpy="0 0 0" />
             <geometry>
-                <mesh filename="file://$(find halfonso_v2)/meshes/right_wheel.stl" />
+                <mesh filename="package://halfonso_v2/meshes/right_wheel.stl" />
             </geometry>
         </collision>
