Commit message: updated config files

File: description/lidar.xacro (robot description, xacro)
@@ -30,5 +30,5 @@
             <origin xyz="0 0 0" rpy="0 0 0" />
             <geometry>
-                <mesh filename="file://$(find halfonso)/meshes/laser_frame.STL" />
+                <mesh filename="file://$(find halfonso_v2)/meshes/laser_frame.STL" />
             </geometry>
             <material name="">
@@ -40,5 +40,5 @@
             <origin xyz="0 0 0" rpy="0 0 0" />
             <geometry>
-                <mesh filename="file://$(find halfonso)/meshes/laser_frame.STL" />
+                <mesh filename="file://$(find halfonso_v2)/meshes/laser_frame.STL" />
             </geometry>
         </collision>

File: description/robot_core.xacro (robot description, xacro)
@@ -65,5 +65,5 @@
             </geometry> -->
             <geometry>
-                <mesh filename="file://$(find halfonso)/meshes/base_footprint.STL" />
+                <mesh filename="file://$(find halfonso_v2)/meshes/base_footprint.STL" />
             </geometry>
             <!-- <material name="orange"/> -->
@@ -82,5 +82,5 @@
             <origin xyz="0 0 0" rpy="0 0 0" />
             <geometry>
-                <mesh filename="file://$(find halfonso)/meshes/base_footprint.STL" />
+                <mesh filename="file://$(find halfonso_v2)/meshes/base_footprint.STL" />
             </geometry>
         </collision>
@@ -118,5 +118,5 @@
             </geometry> -->
             <geometry>
-                <mesh filename="file://$(find halfonso)/meshes/base_link.STL" />
+                <mesh filename="file://$(find halfonso_v2)/meshes/base_link.STL" />
             </geometry>
             <!-- <material name="orange"/> -->
@@ -136,5 +136,5 @@
             <origin xyz="0 0 0" rpy="0 0 0" />
             <geometry>
-                <mesh filename="file://$(find halfonso)/meshes/base_link.STL" />
+                <mesh filename="file://$(find halfonso_v2)/meshes/base_link.STL" />
             </geometry>
         </collision>
@@ -174,5 +174,5 @@
             <geometry>
                 <!-- <cylinder radius="${wheel_radius}" length="${wheel_thickness}"/> -->
-                <mesh filename="file://$(find halfonso)/meshes/left_wheel.STL" />
+                <mesh filename="file://$(find halfonso_v2)/meshes/left_wheel.STL" />
             </geometry>
             <!-- <material name="blue"/> -->
@@ -185,5 +185,5 @@
             <geometry>
                 <!-- <sphere radius="${wheel_radius}"/> -->
-                <mesh filename="file://$(find halfonso)/meshes/left_wheel.STL" />
+                <mesh filename="file://$(find halfonso_v2)/meshes/left_wheel.STL" />
             </geometry>
         </collision>
@@ -221,5 +221,5 @@
             <origin xyz="0 0 0" rpy="0 0 0" />
             <geometry>
-                <mesh filename="file://$(find halfonso)/meshes/right_wheel.STL" />
+                <mesh filename="file://$(find halfonso_v2)/meshes/right_wheel.STL" />
             </geometry>
             <!-- <material name="blue"/> -->
@@ -231,5 +231,5 @@
             <origin xyz="0 0 0" rpy="0 0 0" />
             <geometry>
-                <mesh filename="file://$(find halfonso)/meshes/right_wheel.STL" />
+                <mesh filename="file://$(find halfonso_v2)/meshes/right_wheel.STL" />
             </geometry>
         </collision>

File: description/ros2_control.xacro (robot description, xacro)
@@ -57,5 +57,5 @@
                 name="gz_ros2_control::GazeboSimROS2ControlPlugin">
                 <parameters>
-                    $(find halfonso)/config/controller_gz_sim.yaml
+                    $(find halfonso_v2)/config/controller_gz_sim.yaml
                 </parameters>
             </plugin>

Commit message: updates

File: description/lidar.xacro (robot description, xacro)
@@ -30,5 +30,5 @@
             <origin xyz="0 0 0" rpy="0 0 0" />
             <geometry>
-                <mesh filename="file://$(find halfonso_v2)/meshes/laser_frame.STL" />
+                <mesh filename="file://$(find halfonso_v2)/meshes/laser_frame.stl" />
             </geometry>
             <material name="">
@@ -40,5 +40,5 @@
             <origin xyz="0 0 0" rpy="0 0 0" />
             <geometry>
-                <mesh filename="file://$(find halfonso_v2)/meshes/laser_frame.STL" />
+                <mesh filename="file://$(find halfonso_v2)/meshes/laser_frame.stl" />
             </geometry>
         </collision>

File: description/robot_core.xacro (robot description, xacro)
@@ -65,5 +65,5 @@
             </geometry> -->
             <geometry>
-                <mesh filename="file://$(find halfonso_v2)/meshes/base_footprint.STL" />
+                <mesh filename="file://$(find halfonso_v2)/meshes/base_footprint.stl" />
             </geometry>
             <!-- <material name="orange"/> -->
@@ -82,5 +82,5 @@
             <origin xyz="0 0 0" rpy="0 0 0" />
             <geometry>
-                <mesh filename="file://$(find halfonso_v2)/meshes/base_footprint.STL" />
+                <mesh filename="file://$(find halfonso_v2)/meshes/base_footprint.stl" />
             </geometry>
         </collision>
@@ -118,5 +118,5 @@
             </geometry> -->
             <geometry>
-                <mesh filename="file://$(find halfonso_v2)/meshes/base_link.STL" />
+                <mesh filename="file://$(find halfonso_v2)/meshes/base_link.stl" />
             </geometry>
             <!-- <material name="orange"/> -->
@@ -136,5 +136,5 @@
             <origin xyz="0 0 0" rpy="0 0 0" />
             <geometry>
-                <mesh filename="file://$(find halfonso_v2)/meshes/base_link.STL" />
+                <mesh filename="file://$(find halfonso_v2)/meshes/base_link.stl" />
             </geometry>
         </collision>
@@ -174,5 +174,5 @@
             <geometry>
                 <!-- <cylinder radius="${wheel_radius}" length="${wheel_thickness}"/> -->
-                <mesh filename="file://$(find halfonso_v2)/meshes/left_wheel.STL" />
+                <mesh filename="file://$(find halfonso_v2)/meshes/left_wheel.stl" />
             </geometry>
             <!-- <material name="blue"/> -->
@@ -185,5 +185,5 @@
             <geometry>
                 <!-- <sphere radius="${wheel_radius}"/> -->
-                <mesh filename="file://$(find halfonso_v2)/meshes/left_wheel.STL" />
+                <mesh filename="file://$(find halfonso_v2)/meshes/left_wheel.stl" />
             </geometry>
         </collision>
@@ -221,5 +221,5 @@
             <origin xyz="0 0 0" rpy="0 0 0" />
             <geometry>
-                <mesh filename="file://$(find halfonso_v2)/meshes/right_wheel.STL" />
+                <mesh filename="file://$(find halfonso_v2)/meshes/right_wheel.stl" />
             </geometry>
             <!-- <material name="blue"/> -->
@@ -231,5 +231,5 @@
             <origin xyz="0 0 0" rpy="0 0 0" />
             <geometry>
-                <mesh filename="file://$(find halfonso_v2)/meshes/right_wheel.STL" />
+                <mesh filename="file://$(find halfonso_v2)/meshes/right_wheel.stl" />
             </geometry>
         </collision>

Commit message: changes to robot visualization

File: description/lidar.xacro (robot description, xacro)
@@ -30,5 +30,5 @@
             <origin xyz="0 0 0" rpy="0 0 0" />
             <geometry>
-                <mesh filename="file://$(find halfonso_v2)/meshes/laser_frame.stl" />
+                <mesh filename="package://halfonso_v2/meshes/laser_frame.stl" />
             </geometry>
             <material name="">
@@ -40,5 +40,5 @@
             <origin xyz="0 0 0" rpy="0 0 0" />
             <geometry>
-                <mesh filename="file://$(find halfonso_v2)/meshes/laser_frame.stl" />
+                <mesh filename="package://halfonso_v2/meshes/laser_frame.stl" />
             </geometry>
         </collision>
